File: NumericDisplays.kicad_sch (KiCad schematic)
At the start: 53 parts, among them J1 Conn_01x06_Pin, J2 Conn_01x06_Pin, U1 74HC595, U2 74HC595

Commit message: Update to 47r resistors
Parts:
- R1, R10, R11, R12, R13, R14, R15, R16, R2, R3, R4, R5, R6, R7, R8, R9: value 51 -> 47r
Changed lines of the file:
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@@
 			)
 		)
-		(property "Value" "51"
+		(property "Value" "47r"
 			(at 186.69 97.79 90)
 			(effects
@@
 			)
 		)
-		(property "Value" "51"
+		(property "Value" "47r"
 			(at 134.62 82.55 90)
 			(effects
@@
 			)
 		)
-		(property "Value" "51"
+		(property "Value" "47r"
 			(at 186.69 82.55 90)
 			(effects
@@
 			)
 		)
-		(property "Value" "51"
+		(property "Value" "47r"
 			(at 134.62 87.63 90)
 			(effects
@@
 			)
 		)
-		(property "Value" "51"
+		(property "Value" "47r"
 			(at 134.62 97.79 90)
 			(effects
@@
 			)
 		)
-		(property "Value" "51"
+		(property "Value" "47r"
 			(at 186.69 92.71 90)
 			(effects
@@
 			)
 		)
-		(property "Value" "51"
+		(property "Value" "47r"
 			(at 186.69 87.63 90)
 			(effects
@@
 			)
 		)
-		(property "Value" "51"
+		(property "Value" "47r"
 			(at 186.69 95.25 90)
 			(effects
@@
 			)
 		)
-		(property "Value" "51"
+		(property "Value" "47r"
 			(at 134.62 80.01 90)
 			(effects
@@
 			)
 		)
-		(property "Value" "51"
+		(property "Value" "47r"
 			(at 134.62 95.25 90)
 			(effects
@@
 			)
 		)
-		(property "Value" "51"
+		(property "Value" "47r"
 			(at 134.62 92.71 90)
 			(effects
@@
 			)
 		)
-		(property "Value" "51"
+		(property "Value" "47r"
 			(at 186.69 90.17 90)
 			(effects
@@
 			)
 		)
-		(property "Value" "51"
+		(property "Value" "47r"
 			(at 186.69 85.09 90)
 			(effects
@@
 			)
 		)
-		(property "Value" "51"
+		(property "Value" "47r"
 			(at 186.69 80.01 90)
 			(effects
@@
 			)
 		)
-		(property "Value" "51"
+		(property "Value" "47r"
 			(at 134.62 90.17 90)
 			(effects
@@
 			)
 		)
-		(property "Value" "51"
+		(property "Value" "47r"
 			(at 134.62 85.09 90)
 			(effects
